File: elec/layout/emmc/emmc.kicad_pcb (KiCad board)
At the start: 2 copper layers, 12 parts, among them U1 _Samsung_KLMBG2JETD_B041

Commit message: update naming
Connections:
- net *2E88-net renamed *6198-net
- net *2E88.eMMC.VDD_INTERNAL-net renamed *6198.eMMC.VDD_INTERNAL-net
- net *2E88.eMMC.footprint.pins[0].net-net renamed *6198.eMMC.footprint.pins[0].net-net
- net *2E88.eMMC.footprint.pins[101].net-net renamed *6198.eMMC.footprint.pins[101].net-net
- net *2E88.eMMC.footprint.pins[102].net-net renamed *6198.eMMC.footprint.pins[102].net-net
- net *2E88.eMMC.footprint.pins[105].net-net renamed *6198.eMMC.footprint.pins[105].net-net
- net *2E88.eMMC.footprint.pins[106].net-net renamed *6198.eMMC.footprint.pins[106].net-net
- net *2E88.eMMC.footprint.pins[107].net-net renamed *6198.eMMC.footprint.pins[107].net-net
- net *2E88.eMMC.footprint.pins[108].net-net renamed *6198.eMMC.footprint.pins[108].net-net
- net *2E88.eMMC.footprint.pins[109].net-net renamed *6198.eMMC.footprint.pins[109].net-net
- net *2E88.eMMC.footprint.pins[110].net-net renamed *6198.eMMC.footprint.pins[110].net-net
- net *2E88.eMMC.footprint.pins[111].net-net renamed *6198.eMMC.footprint.pins[111].net-net
- net *2E88.eMMC.footprint.pins[112].net-net renamed *6198.eMMC.footprint.pins[112].net-net
- net *2E88.eMMC.footprint.pins[113].net-net renamed *6198.eMMC.footprint.pins[113].net-net
- net *2E88.eMMC.footprint.pins[114].net-net renamed *6198.eMMC.footprint.pins[114].net-net
- net *2E88.eMMC.footprint.pins[115].net-net renamed *6198.eMMC.footprint.pins[115].net-net
- net *2E88.eMMC.footprint.pins[116].net-net renamed *6198.eMMC.footprint.pins[116].net-net
- net *2E88.eMMC.footprint.pins[117].net-net renamed *6198.eMMC.footprint.pins[117].net-net
- net *2E88.eMMC.footprint.pins[118].net-net renamed *6198.eMMC.footprint.pins[118].net-net
- net *2E88.eMMC.footprint.pins[11].net-net renamed *6198.eMMC.footprint.pins[11].net-net
- net *2E88.eMMC.footprint.pins[122].net-net renamed *6198.eMMC.footprint.pins[122].net-net
- net *2E88.eMMC.footprint.pins[123].net-net renamed *6198.eMMC.footprint.pins[123].net-net
- net *2E88.eMMC.footprint.pins[124].net-net renamed *6198.eMMC.footprint.pins[124].net-net
- net *2E88.eMMC.footprint.pins[125].net-net renamed *6198.eMMC.footprint.pins[125].net-net
- net *2E88.eMMC.footprint.pins[126].net-net renamed *6198.eMMC.footprint.pins[126].net-net
- net *2E88.eMMC.footprint.pins[127].net-net renamed *6198.eMMC.footprint.pins[127].net-net
- net *2E88.eMMC.footprint.pins[128].net-net renamed *6198.eMMC.footprint.pins[128].net-net
- net *2E88.eMMC.footprint.pins[129].net-net renamed *6198.eMMC.footprint.pins[129].net-net
- net *2E88.eMMC.footprint.pins[12].net-net renamed *6198.eMMC.footprint.pins[12].net-net
- net *2E88.eMMC.footprint.pins[130].net-net renamed *6198.eMMC.footprint.pins[130].net-net
- net *2E88.eMMC.footprint.pins[132].net-net renamed *6198.eMMC.footprint.pins[132].net-net
- net *2E88.eMMC.footprint.pins[135].net-net renamed *6198.eMMC.footprint.pins[135].net-net
- net *2E88.eMMC.footprint.pins[136].net-net renamed *6198.eMMC.footprint.pins[136].net-net
- net *2E88.eMMC.footprint.pins[137].net-net renamed *6198.eMMC.footprint.pins[137].net-net
- net *2E88.eMMC.footprint.pins[138].net-net renamed *6198.eMMC.footprint.pins[138].net-net
- net *2E88.eMMC.footprint.pins[139].net-net renamed *6198.eMMC.footprint.pins[139].net-net
- net *2E88.eMMC.footprint.pins[13].net-net renamed *6198.eMMC.footprint.pins[13].net-net
- net *2E88.eMMC.footprint.pins[140].net-net renamed *6198.eMMC.footprint.pins[140].net-net
- net *2E88.eMMC.footprint.pins[141].net-net renamed *6198.eMMC.footprint.pins[141].net-net
- net *2E88.eMMC.footprint.pins[142].net-net renamed *6198.eMMC.footprint.pins[142].net-net
- net *2E88.eMMC.footprint.pins[143].net-net renamed *6198.eMMC.footprint.pins[143].net-net
- net *2E88.eMMC.footprint.pins[144].net-net renamed *6198.eMMC.footprint.pins[144].net-net
- net *2E88.eMMC.footprint.pins[145].net-net renamed *6198.eMMC.footprint.pins[145].net-net
- net *2E88.eMMC.footprint.pins[14].net-net renamed *6198.eMMC.footprint.pins[14].net-net
- net *2E88.eMMC.footprint.pins[150].net-net renamed *6198.eMMC.footprint.pins[150].net-net
- net *2E88.eMMC.footprint.pins[151].net-net renamed *6198.eMMC.footprint.pins[151].net-net
- net *2E88.eMMC.footprint.pins[152].net-net renamed *6198.eMMC.footprint.pins[152].net-net
- net *2E88.eMMC.footprint.pins[15].net-net renamed *6198.eMMC.footprint.pins[15].net-net
- net *2E88.eMMC.footprint.pins[16].net-net renamed *6198.eMMC.footprint.pins[16].net-net
- net *2E88.eMMC.footprint.pins[17].net-net renamed *6198.eMMC.footprint.pins[17].net-net
- net *2E88.eMMC.footprint.pins[18].net-net renamed *6198.eMMC.footprint.pins[18].net-net
- net *2E88.eMMC.footprint.pins[19].net-net renamed *6198.eMMC.footprint.pins[19].net-net
- net *2E88.eMMC.footprint.pins[1].net-net renamed *6198.eMMC.footprint.pins[1].net-net
- net *2E88.eMMC.footprint.pins[25].net-net renamed *6198.eMMC.footprint.pins[25].net-net
- net *2E88.eMMC.footprint.pins[26].net-net renamed *6198.eMMC.footprint.pins[26].net-net
- net *2E88.eMMC.footprint.pins[27].net-net renamed *6198.eMMC.footprint.pins[27].net-net
- net *2E88.eMMC.footprint.pins[28].net-net renamed *6198.eMMC.footprint.pins[28].net-net
- net *2E88.eMMC.footprint.pins[29].net-net renamed *6198.eMMC.footprint.pins[29].net-net
- net *2E88.eMMC.footprint.pins[2].net-net renamed *6198.eMMC.footprint.pins[2].net-net
- net *2E88.eMMC.footprint.pins[30].net-net renamed *6198.eMMC.footprint.pins[30].net-net
- net *2E88.eMMC.footprint.pins[31].net-net renamed *6198.eMMC.footprint.pins[31].net-net
- net *2E88.eMMC.footprint.pins[32].net-net renamed *6198.eMMC.footprint.pins[32].net-net
- net *2E88.eMMC.footprint.pins[33].net-net renamed *6198.eMMC.footprint.pins[33].net-net
- net *2E88.eMMC.footprint.pins[35].net-net renamed *6198.eMMC.footprint.pins[35].net-net
- net *2E88.eMMC.footprint.pins[37].net-net renamed *6198.eMMC.footprint.pins[37].net-net
- net *2E88.eMMC.footprint.pins[39].net-net renamed *6198.eMMC.footprint.pins[39].net-net
- net *2E88.eMMC.footprint.pins[3].net-net renamed *6198.eMMC.footprint.pins[3].net-net
- net *2E88.eMMC.footprint.pins[40].net-net renamed *6198.eMMC.footprint.pins[40].net-net
- net *2E88.eMMC.footprint.pins[41].net-net renamed *6198.eMMC.footprint.pins[41].net-net
- net *2E88.eMMC.footprint.pins[42].net-net renamed *6198.eMMC.footprint.pins[42].net-net
- net *2E88.eMMC.footprint.pins[43].net-net renamed *6198.eMMC.footprint.pins[43].net-net
- net *2E88.eMMC.footprint.pins[44].net-net renamed *6198.eMMC.footprint.pins[44].net-net
- net *2E88.eMMC.footprint.pins[45].net-net renamed *6198.eMMC.footprint.pins[45].net-net
- net *2E88.eMMC.footprint.pins[46].net-net renamed *6198.eMMC.footprint.pins[46].net-net
- net *2E88.eMMC.footprint.pins[47].net-net renamed *6198.eMMC.footprint.pins[47].net-net
- net *2E88.eMMC.footprint.pins[48].net-net renamed *6198.eMMC.footprint.pins[48].net-net
- net *2E88.eMMC.footprint.pins[49].net-net renamed *6198.eMMC.footprint.pins[49].net-net
- net *2E88.eMMC.footprint.pins[4].net-net renamed *6198.eMMC.footprint.pins[4].net-net
- net *2E88.eMMC.footprint.pins[50].net-net renamed *6198.eMMC.footprint.pins[50].net-net
- net *2E88.eMMC.footprint.pins[51].net-net renamed *6198.eMMC.footprint.pins[51].net-net
- net *2E88.eMMC.footprint.pins[52].net-net renamed *6198.eMMC.footprint.pins[52].net-net
- net *2E88.eMMC.footprint.pins[53].net-net renamed *6198.eMMC.footprint.pins[53].net-net
- net *2E88.eMMC.footprint.pins[54].net-net renamed *6198.eMMC.footprint.pins[54].net-net
- net *2E88.eMMC.footprint.pins[55].net-net renamed *6198.eMMC.footprint.pins[55].net-net
- net *2E88.eMMC.footprint.pins[56].net-net renamed *6198.eMMC.footprint.pins[56].net-net
- net *2E88.eMMC.footprint.pins[59].net-net renamed *6198.eMMC.footprint.pins[59].net-net
- net *2E88.eMMC.footprint.pins[5].net-net renamed *6198.eMMC.footprint.pins[5].net-net
- net *2E88.eMMC.footprint.pins[60].net-net renamed *6198.eMMC.footprint.pins[60].net-net
- net *2E88.eMMC.footprint.pins[61].net-net renamed *6198.eMMC.footprint.pins[61].net-net
- net *2E88.eMMC.footprint.pins[62].net-net renamed *6198.eMMC.footprint.pins[62].net-net
- net *2E88.eMMC.footprint.pins[63].net-net renamed *6198.eMMC.footprint.pins[63].net-net
- net *2E88.eMMC.footprint.pins[64].net-net renamed *6198.eMMC.footprint.pins[64].net-net
- net *2E88.eMMC.footprint.pins[65].net-net renamed *6198.eMMC.footprint.pins[65].net-net
- net *2E88.eMMC.footprint.pins[66].net-net renamed *6198.eMMC.footprint.pins[66].net-net
- net *2E88.eMMC.footprint.pins[67].net-net renamed *6198.eMMC.footprint.pins[67].net-net
- net *2E88.eMMC.footprint.pins[69].net-net renamed *6198.eMMC.footprint.pins[69].net-net
- net *2E88.eMMC.footprint.pins[6].net-net renamed *6198.eMMC.footprint.pins[6].net-net
- net *2E88.eMMC.footprint.pins[70].net-net renamed *6198.eMMC.footprint.pins[70].net-net
- net *2E88.eMMC.footprint.pins[71].net-net renamed *6198.eMMC.footprint.pins[71].net-net
- net *2E88.eMMC.footprint.pins[72].net-net renamed *6198.eMMC.footprint.pins[72].net-net
- net *2E88.eMMC.footprint.pins[73].net-net renamed *6198.eMMC.footprint.pins[73].net-net
- net *2E88.eMMC.footprint.pins[74].net-net renamed *6198.eMMC.footprint.pins[74].net-net
- net *2E88.eMMC.footprint.pins[75].net-net renamed *6198.eMMC.footprint.pins[75].net-net
- net *2E88.eMMC.footprint.pins[77].net-net renamed *6198.eMMC.footprint.pins[77].net-net
- net *2E88.eMMC.footprint.pins[79].net-net renamed *6198.eMMC.footprint.pins[79].net-net
- net *2E88.eMMC.footprint.pins[80].net-net renamed *6198.eMMC.footprint.pins[80].net-net
- net *2E88.eMMC.footprint.pins[81].net-net renamed *6198.eMMC.footprint.pins[81].net-net
- net *2E88.eMMC.footprint.pins[82].net-net renamed *6198.eMMC.footprint.pins[82].net-net
- net *2E88.eMMC.footprint.pins[83].net-net renamed *6198.eMMC.footprint.pins[83].net-net
- net *2E88.eMMC.footprint.pins[85].net-net renamed *6198.eMMC.footprint.pins[85].net-net
- net *2E88.eMMC.footprint.pins[87].net-net renamed *6198.eMMC.footprint.pins[87].net-net
- net *2E88.eMMC.footprint.pins[88].net-net renamed *6198.eMMC.footprint.pins[88].net-net
- net *2E88.eMMC.footprint.pins[89].net-net renamed *6198.eMMC.footprint.pins[89].net-net
- net *2E88.eMMC.footprint.pins[90].net-net renamed *6198.eMMC.footprint.pins[90].net-net
- net *2E88.eMMC.footprint.pins[91].net-net renamed *6198.eMMC.footprint.pins[91].net-net
- net *2E88.eMMC.footprint.pins[93].net-net renamed *6198.eMMC.footprint.pins[93].net-net
- net *2E88.eMMC.footprint.pins[94].net-net renamed *6198.eMMC.footprint.pins[94].net-net
- net *2E88.eMMC.footprint.pins[95].net-net renamed *6198.eMMC.footprint.pins[95].net-net
- net *2E88.eMMC.footprint.pins[96].net-net renamed *6198.eMMC.footprint.pins[96].net-net
- net *2E88.eMMC.footprint.pins[97].net-net renamed *6198.eMMC.footprint.pins[97].net-net
- net *2E88.eMMC.footprint.pins[98].net-net renamed *6198.eMMC.footprint.pins[98].net-net
- net *2E88.eMMC.footprint.pins[99].net-net renamed *6198.eMMC.footprint.pins[99].net-net
