File: elec/layout/cm4/cm4.kicad_pcb (KiCad board)
At the start: 2 copper layers, 4 parts, among them CN1 HRSHirose_DF40C_100DS_0_4V51, CN2 HRSHirose_DF40C_100DS_0_4V51, U1 _Texas_Instruments_SN74LVC1G0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

Commit message: rename pdcontroller folder
Connections:
- CN1 pad 12: signal-9 -> pins[23]
- CN1 pad 14: pins[27] -> signal-13
- CN1 pad 15: signal-3 -> signal-11
- CN1 pad 19: pins[37] -> signal-3
- CN1 pad 23: pins[45] -> signal
- CN1 pad 24: pins[47] -> signal-4
- CN1 pad 27: signal -> pins[53]
- CN1 pad 28: pins[55] -> signal-2
- CN1 pad 73: signal-11 -> signal-10
- CN1 pad 75: signal-6 -> signal-5
- CN1 pad 77: signal-10 -> signal-9
- CN1 pad 78: signal-1 -> pins[44]
- CN1 pad 80: signal-2 -> pins[40]
- CN1 pad 81: signal-4 -> signal-1
- CN1 pad 82: signal-5 -> pins[36]
- CN1 pad 85: pins[30] -> signal-6
- CN1 pad 87: pins[26] -> signal-12
- CN2 pad 12: pins[23] -> hdi_b-pins[23]
- CN2 pad 14: hdi_b-pins[27] -> pins[27]
- CN2 pad 78: pins[44] -> pins[44]-1
- CN2 pad 80: pins[40] -> hdi_b-pins[40]
- CN2 pad 87: hdi_b-pins[26] -> pins[26]
Changed lines of the file:
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@@
     (net 3 "pins[49]")
     (net 4 "pins[44]")
-    (net 5 "pins[47]")
+    (net 5 "pins[44]-1")
     (net 6 "hdi_b-pins[62]")
     (net 7 "USB2_D_N")
@@
     (net 19 "ETH_P1_P")
     (net 20 "pins[18]")
-    (net 21 "hdi_b-pins[27]")
-    (net 22 "pins[30]")
+    (net 21 "signal-13")
+    (net 22 "hdi_b-pins[23]")
     (net 23 "hdi_a-pins[34]")
     (net 24 "pins[67]")
@@
     (net 80 "HDMI1_D2_P")
     (net 81 "pins[95]")
-    (net 82 "pins[37]")
+    (net 82 "pins[36]")
     (net 83 "hdi_a-pins[17]")
     (net 84 "HDMI1_CK_N")
@@
     (net 106 "hdi_b-pins[92]")
     (net 107 "ETH_LED_LINK")
-    (net 108 "pins[45]")
+    (net 108 "hdi_b-pins[40]")
     (net 109 "pins[63]")
     (net 110 "ETH_P1_N")
@@
     (net 112 "signal-5")
     (net 113 "hdi_a-pins[94]")
-    (net 114 "pins[55]")
+    (net 114 "pins[53]")
     (net 115 "signal-3")
-    (net 116 "hdi_b-pins[26]")
+    (net 116 "signal-12")
     (net 117 "ETH_P0_P")
     (net 118 "HDMI1_D0_N")
@@
             (layers "F.Cu" "F.Paste" "F.Mask")
             (remove_unused_layers no)
-            (net 57 "pins[23]")
+            (net 22 "hdi_b-pins[23]")
 )
         (pad "13" smd rect
@@
             (layers "F.Cu" "F.Paste" "F.Mask")
             (remove_unused_layers no)
-            (net 21 "hdi_b-pins[27]")
+            (net 28 "pins[27]")
 )
         (pad "15" smd rect
@@
             (layers "F.Cu" "F.Paste" "F.Mask")
             (remove_unused_layers no)
-            (net 4 "pins[44]")
+            (net 5 "pins[44]-1")
 )
         (pad "79" smd rect
@@
             (layers "F.Cu" "F.Paste" "F.Mask")
             (remove_unused_layers no)
-            (net 89 "pins[40]")
+            (net 108 "hdi_b-pins[40]")
 )
         (pad "81" smd rect
@@
             (layers "F.Cu" "F.Paste" "F.Mask")
             (remove_unused_layers no)
-            (net 116 "hdi_b-pins[26]")
+            (net 73 "pins[26]")
 )
         (pad "88" smd rect
@@
             (layers "F.Cu" "F.Paste" "F.Mask")
             (remove_unused_layers no)
-            (net 99 "signal-9")
+            (net 57 "pins[23]")
 )
         (pad "13" smd rect
@@
             (layers "F.Cu" "F.Paste" "F.Mask")
             (remove_unused_layers no)
-            (net 28 "pins[27]")
+            (net 21 "signal-13")
 )
         (pad "15" smd rect
@@
             (layers "F.Cu" "F.Paste" "F.Mask")
             (remove_unused_layers no)
-            (net 115 "signal-3")
+            (net 102 "signal-11")
 )
         (pad "16" smd rect
@@
             (layers "F.Cu" "F.Paste" "F.Mask")
             (remove_unused_layers no)
-            (net 82 "pins[37]")
+            (net 115 "signal-3")
 )
         (pad "20" smd rect
@@
             (layers "F.Cu" "F.Paste" "F.Mask")
             (remove_unused_layers no)
-            (net 108 "pins[45]")
+            (net 12 "signal")
 )
         (pad "24" smd rect
@@
             (layers "F.Cu" "F.Paste" "F.Mask")
             (remove_unused_layers no)
-            (net 5 "pins[47]")
+            (net 36 "signal-4")
 )
         (pad "25" smd rect
@@
             (layers "F.Cu" "F.Paste" "F.Mask")
             (remove_unused_layers no)
-            (net 12 "signal")
+            (net 114 "pins[53]")
 )
         (pad "28" smd rect
@@
             (layers "F.Cu" "F.Paste" "F.Mask")
             (remove_unused_layers no)
-            (net 114 "pins[55]")
+            (net 26 "signal-2")
 )
         (pad "29" smd rect
@@
             (layers "F.Cu" "F.Paste" "F.Mask")
             (remove_unused_layers no)
-            (net 102 "signal-11")
+            (net 70 "signal-10")
 )
         (pad "74" smd rect
@@
             (layers "F.Cu" "F.Paste" "F.Mask")
             (remove_unused_layers no)
-            (net 18 "signal-6")
+            (net 112 "signal-5")
 )
         (pad "76" smd rect
@@
             (layers "F.Cu" "F.Paste" "F.Mask")
             (remove_unused_layers no)
-            (net 70 "signal-10")
+            (net 99 "signal-9")
 )
         (pad "78" smd rect
@@
             (layers "F.Cu" "F.Paste" "F.Mask")
             (remove_unused_layers no)
-            (net 10 "signal-1")
+            (net 4 "pins[44]")
 )
         (pad "79" smd rect
@@
             (layers "F.Cu" "F.Paste" "F.Mask")
             (remove_unused_layers no)
-            (net 26 "signal-2")
+            (net 89 "pins[40]")
 )
         (pad "81" smd rect
@@
             (layers "F.Cu" "F.Paste" "F.Mask")
             (remove_unused_layers no)
-            (net 36 "signal-4")
+            (net 10 "signal-1")
 )
         (pad "82" smd rect
@@
             (layers "F.Cu" "F.Paste" "F.Mask")
             (remove_unused_layers no)
-            (net 112 "signal-5")
+            (net 82 "pins[36]")
 )
         (pad "83" smd rect
@@
             (layers "F.Cu" "F.Paste" "F.Mask")
             (remove_unused_layers no)
-            (net 22 "pins[30]")
+            (net 18 "signal-6")
 )
         (pad "86" smd rect
@@
             (layers "F.Cu" "F.Paste" "F.Mask")
             (remove_unused_layers no)
-            (net 73 "pins[26]")
+            (net 116 "signal-12")
 )
         (pad "88" smd rect

Commit message: layout sync working
Connections:
- net signal-10 renamed pins[54]
- net signal-6 renamed pins[30]
- net signal-7 renamed pins[57]
- CN1 pad 12: pins[23] -> signal-5
- CN1 pad 14: signal-13 -> pins[27]
- CN1 pad 15: signal-11 -> pins[29]
- CN1 pad 19: signal-3 -> pins[37]
- CN1 pad 20: pins[39] -> signal-3
- CN1 pad 22: pins[43] -> signal-1
- CN1 pad 23: signal -> pins[45]
- CN1 pad 24: signal-4 -> signal
- CN1 pad 25: signal-8 -> pins[49]
- CN1 pad 28: signal-2 -> signal-4
- CN1 pad 75: signal-5 -> pins[50]
- CN1 pad 77: signal-9 -> pins[46]
- CN1 pad 81: signal-1 -> pins[38]
- CN1 pad 86: pins[28] -> signal-2
- CN1 pad 87: signal-12 -> pins[26]
- CN2 pad 12: hdi_b-pins[23] -> pins[23]
- CN2 pad 14: pins[27] -> hdi_b-pins[27]
- CN2 pad 15: pins[29] -> hdi_b-pins[29]
- CN2 pad 20: hdi_b-pins[39] -> pins[39]
- CN2 pad 25: pins[49] -> hdi_b-pins[49]
- CN2 pad 77: pins[46] -> pins[46]-1
- CN2 pad 81: pins[38] -> hdi_b-pins[38]
- CN2 pad 86: hdi_b-pins[28] -> pins[28]
- CN2 pad 87: pins[26] -> hdi_b-pins[26]
Changed lines of the file:
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@@
     (net 3 "pins[49]")
     (net 4 "pins[44]")
-    (net 5 "pins[44]-1")
+    (net 5 "hdi_b-pins[26]")
     (net 6 "hdi_b-pins[62]")
     (net 7 "USB2_D_N")
@@
     (net 16 "hdi_a-pins[62]")
     (net 17 "pins[32]")
-    (net 18 "signal-6")
+    (net 18 "pins[53]")
     (net 19 "ETH_P1_P")
     (net 20 "pins[18]")
-    (net 21 "signal-13")
-    (net 22 "hdi_b-pins[23]")
+    (net 21 "hdi_b-pins[27]")
+    (net 22 "pins[46]-1")
     (net 23 "hdi_a-pins[34]")
     (net 24 "pins[67]")
@@
     (net 32 "VCC_5V")
     (net 33 "hdi_b-pins[68]")
-    (net 34 "hdi_b-pins[39]")
+    (net 34 "pins[54]")
     (net 35 "pins[98]")
     (net 36 "signal-4")
@@
     (net 59 "n_c_")
     (net 60 "pins[90]")
-    (net 61 "signal-7")
+    (net 61 "hdi_b-pins[40]")
     (net 62 "pins[82]")
     (net 63 "HDMI0_D2_P")
@@
     (net 68 "pins[58]")
     (net 69 "hdi_a-pins[93]")
-    (net 70 "signal-10")
+    (net 70 "pins[57]")
     (net 71 "HDMI1_D2_N")
     (net 72 "HDMI0_D0_P")
     (net 73 "pins[26]")
-    (net 74 "pins[43]")
+    (net 74 "pins[44]-1")
     (net 75 "pins[39]")
     (net 76 "pins[76]")
@@
     (net 96 "HDMI0_D0_N")
     (net 97 "HDMI1_D0_P")
-    (net 98 "hdi_b-pins[28]")
-    (net 99 "signal-9")
+    (net 98 "hdi_b-pins[33]")
+    (net 99 "pins[30]")
     (net 100 "pins[66]")
     (net 101 "pins[41]")
-    (net 102 "signal-11")
+    (net 102 "pins[50]")
     (net 103 "pins[91]")
     (net 104 "hdi_b-pins[88]")
@@
     (net 106 "hdi_b-pins[92]")
     (net 107 "ETH_LED_LINK")
-    (net 108 "hdi_b-pins[40]")
+    (net 108 "pins[37]")
     (net 109 "pins[63]")
     (net 110 "ETH_P1_N")
@@
     (net 112 "signal-5")
     (net 113 "hdi_a-pins[94]")
-    (net 114 "pins[53]")
+    (net 114 "hdi_b-pins[29]")
     (net 115 "signal-3")
-    (net 116 "signal-12")
+    (net 116 "hdi_b-pins[49]")
     (net 117 "ETH_P0_P")
     (net 118 "HDMI1_D0_N")
@@
     (net 130 "hdi_b-pins[15]")
     (net 131 "pins[3]")
-    (net 132 "hdi_b-pins[33]")
+    (net 132 "hdi_b-pins[38]")
     (net 133 "pins[71]")
     (net 134 "pins[21]")
@@
     (net 141 "pins[38]")
     (net 142 "hdi_a-pins[15]")
-    (net 143 "signal-8")
+    (net 143 "pins[45]")
     (net 144 "HDMI0_D1_P")
     (net 145 "HDMI1_HOTPLUG")
@@
             (layers "F.Cu" "F.Paste" "F.Mask")
             (remove_unused_layers no)
-            (net 22 "hdi_b-pins[23]")
+            (net 57 "pins[23]")
 )
         (pad "13" smd rect
@@
             (layers "F.Cu" "F.Paste" "F.Mask")
             (remove_unused_layers no)
-            (net 28 "pins[27]")
+            (net 21 "hdi_b-pins[27]")
 )
         (pad "15" smd rect
@@
             (layers "F.Cu" "F.Paste" "F.Mask")
             (remove_unused_layers no)
-            (net 64 "pins[29]")
+            (net 114 "hdi_b-pins[29]")
 )
         (pad "16" smd rect
@@
             (layers "F.Cu" "F.Paste" "F.Mask")
             (remove_unused_layers no)
-            (net 132 "hdi_b-pins[33]")
+            (net 98 "hdi_b-pins[33]")
 )
         (pad "18" smd rect
@@
             (layers "F.Cu" "F.Paste" "F.Mask")
             (remove_unused_layers no)
-            (net 34 "hdi_b-pins[39]")
+            (net 75 "pins[39]")
 )
         (pad "21" smd rect
@@
             (layers "F.Cu" "F.Paste" "F.Mask")
             (remove_unused_layers no)
-            (net 3 "pins[49]")
+            (net 116 "hdi_b-pins[49]")
 )
         (pad "26" smd rect
@@
             (layers "F.Cu" "F.Paste" "F.Mask")
             (remove_unused_layers no)
-            (net 9 "pins[46]")
+            (net 22 "pins[46]-1")
 )
         (pad "78" smd rect
@@
             (layers "F.Cu" "F.Paste" "F.Mask")
             (remove_unused_layers no)
-            (net 5 "pins[44]-1")
+            (net 74 "pins[44]-1")
 )
         (pad "79" smd rect
@@
             (layers "F.Cu" "F.Paste" "F.Mask")
             (remove_unused_layers no)
-            (net 108 "hdi_b-pins[40]")
+            (net 61 "hdi_b-pins[40]")
 )
         (pad "81" smd rect
@@
             (layers "F.Cu" "F.Paste" "F.Mask")
             (remove_unused_layers no)
-            (net 141 "pins[38]")
+            (net 132 "hdi_b-pins[38]")
 )
         (pad "82" smd rect
@@
             (layers "F.Cu" "F.Paste" "F.Mask")
             (remove_unused_layers no)
-            (net 98 "hdi_b-pins[28]")
+            (net 139 "pins[28]")
 )
         (pad "87" smd rect
@@
             (layers "F.Cu" "F.Paste" "F.Mask")
             (remove_unused_layers no)
-            (net 73 "pins[26]")
+            (net 5 "hdi_b-pins[26]")
 )
         (pad "88" smd rect
@@
             (layers "F.Cu" "F.Paste" "F.Mask")
             (remove_unused_layers no)
-            (net 57 "pins[23]")
+            (net 112 "signal-5")
 )
         (pad "13" smd rect
@@
             (layers "F.Cu" "F.Paste" "F.Mask")
             (remove_unused_layers no)
-            (net 21 "signal-13")
+            (net 28 "pins[27]")
 )
         (pad "15" smd rect
@@
             (layers "F.Cu" "F.Paste" "F.Mask")
             (remove_unused_layers no)
-            (net 102 "signal-11")
+            (net 64 "pins[29]")
 )
         (pad "16" smd rect
@@
             (layers "F.Cu" "F.Paste" "F.Mask")
             (remove_unused_layers no)
-            (net 115 "signal-3")
+            (net 108 "pins[37]")
 )
         (pad "20" smd rect
@@
             (layers "F.Cu" "F.Paste" "F.Mask")
             (remove_unused_layers no)
-            (net 75 "pins[39]")
+            (net 115 "signal-3")
 )
         (pad "21" smd rect
@@
             (layers "F.Cu" "F.Paste" "F.Mask")
             (remove_unused_layers no)
-            (net 74 "pins[43]")
+            (net 10 "signal-1")
 )
         (pad "23" smd rect
@@
             (layers "F.Cu" "F.Paste" "F.Mask")
             (remove_unused_layers no)
-            (net 12 "signal")
+            (net 143 "pins[45]")
 )
         (pad "24" smd rect
@@
             (layers "F.Cu" "F.Paste" "F.Mask")
             (remove_unused_layers no)
-            (net 36 "signal-4")
+            (net 12 "signal")
 )
         (pad "25" smd rect
@@
             (layers "F.Cu" "F.Paste" "F.Mask")
             (remove_unused_layers no)
-            (net 143 "signal-8")
+            (net 3 "pins[49]")
 )
         (pad "26" smd rect
@@
             (layers "F.Cu" "F.Paste" "F.Mask")
             (remove_unused_layers no)
-            (net 114 "pins[53]")
+            (net 18 "pins[53]")
 )
         (pad "28" smd rect
@@
             (layers "F.Cu" "F.Paste" "F.Mask")
             (remove_unused_layers no)
-            (net 26 "signal-2")
+            (net 36 "signal-4")
 )
         (pad "29" smd rect
@@
             (layers "F.Cu" "F.Paste" "F.Mask")
             (remove_unused_layers no)
-            (net 61 "signal-7")
+            (net 70 "pins[57]")
 )
         (pad "30" smd rect
@@
             (layers "F.Cu" "F.Paste" "F.Mask")
             (remove_unused_layers no)
-            (net 70 "signal-10")
+            (net 34 "pins[54]")
 )
         (pad "74" smd rect
@@
             (layers "F.Cu" "F.Paste" "F.Mask")
             (remove_unused_layers no)
-            (net 112 "signal-5")
+            (net 102 "pins[50]")
 )
         (pad "76" smd rect
@@
             (layers "F.Cu" "F.Paste" "F.Mask")
             (remove_unused_layers no)
-            (net 99 "signal-9")
+            (net 9 "pins[46]")
 )
         (pad "78" smd rect
@@
             (layers "F.Cu" "F.Paste" "F.Mask")
             (remove_unused_layers no)
-            (net 10 "signal-1")
+            (net 141 "pins[38]")
 )
         (pad "82" smd rect
@@
             (layers "F.Cu" "F.Paste" "F.Mask")
             (remove_unused_layers no)
-            (net 18 "signal-6")
+            (net 99 "pins[30]")
 )
         (pad "86" smd rect
@@
             (layers "F.Cu" "F.Paste" "F.Mask")
             (remove_unused_layers no)
-            (net 139 "pins[28]")
+            (net 26 "signal-2")
 )
         (pad "87" smd rect
@@
             (layers "F.Cu" "F.Paste" "F.Mask")
             (remove_unused_layers no)
-            (net 116 "signal-12")
+            (net 73 "pins[26]")
 )
         (pad "88" smd rect
