File: elec/layout/pd-controller.kicad_pcb (KiCad board)
At the start: 2 copper layers, 0 parts

Commit message: builds working
Parts:
- added C1: 4.7µF ±10% 35V X5R, lcsc:C0603, F.Cu at (132.8, 99.2)
- added C2: 100nF ±10% 10V X5R, lcsc:C0201, F.Cu at (142.3, 105.2)
- added C3: 1µF ±20% 6.3V X5R, lcsc:C0201, F.Cu at (139.5, 104.9)
- added C4: 1µF ±20% 6.3V X5R, lcsc:C0201, F.Cu at (138.5, 104.8)
- added D1: ESDA25W, lcsc:SOT-323-3_L2.1-W1.3-P1.32-LS2.1-BR, F.Cu at (136.0, 105.3)
- added D2: , lcsc:DFN1610-2_L1.6-W1.0-P1.05-RD, F.Cu at (135.6, 99.9)
- added D3: , lcsc:DFN1610-2_L1.6-W1.0-P1.05-RD, F.Cu at (138.6, 99.9)
- added Q1: MOSFET, lcsc:SOT-23-3_L2.9-W1.3-P1.90-LS2.4-BR-1, F.Cu at (136.5, 102.4)
- added R1: 1kΩ ±1% 50mW, lcsc:R0201, F.Cu at (139.3, 111.4)
- added R2: 4.7kΩ ±1% 50mW, lcsc:R0201, F.Cu at (137.2, 111.4)
- added R3: 4.7kΩ ±1% 50mW, lcsc:R0201, F.Cu at (138.2, 111.4)
- added R4: 1kΩ ±1% 50mW, lcsc:R0201, F.Cu at (141.1, 105.1)
- added R5: 100kΩ ±1% 50mW, lcsc:R0201, F.Cu at (142.9, 106.3)
- added R6: 22.1kΩ ±1% 50mW, lcsc:R0201, F.Cu at (142.3, 107.4)
- added R7: 100Ω ±1% 50mW, lcsc:R0201, F.Cu at (142.3, 106.3)
- added U1: STUSB4500QTR, lcsc:QFN-24_L4.0-W4.0-P0.50-BL-EP2.8, F.Cu at (139.1, 108.1)
- added U2: _HCTL_HC_TYPE_C_24P_VS9_3_5A_F1_1_04, lcsc:USB-C-SMD_HC-TYPE-C-24P-VS9.3-5A-F1.1-04, B.Cu at (156.1, 111.4)
