File: elec/layout/capacitive-sensor.kicad_pcb (KiCad board)
At the start: 2 copper layers, 7 parts, among them U1 _Microchip_Tech_CAP1188_1_CP_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

Commit message: refactor PD controller + remove params
Parts:
- removed C1: 100nF ±10% 16V X7R, lcsc:C0402
- removed R1, R4, R5: 10kΩ ±1% 62.5mW, lcsc:R0402
- removed R2, R3: 5.1kΩ ±1% 62.5mW, lcsc:R0402
- removed U1: _Microchip_Tech_CAP1188_1_CP_TR, lcsc:QFN-24_L4.0-W4.0-P0.50-TL-EP2.5

Commit message: Build full
Parts:
- added C1: 100nF ±10% 50V X7R, lcsc:C0603, F.Cu at (10.0, 0.00)
- added R1: 10kΩ ±1% 62.5mW, lcsc:R0402, F.Cu at (20.0, 0.00)
- added R2: 10kΩ ±1% 62.5mW, lcsc:R0402, F.Cu at (30.0, 0.00)
- added R3: 10kΩ ±1% 62.5mW, lcsc:R0402, F.Cu at (40.0, 0.00)
- added R4: 1kΩ ±1% 100mW, lcsc:R0603, F.Cu at (50.0, 0.00)
- added R5: 1kΩ ±1% 100mW, lcsc:R0603, F.Cu at (60.0, 0.00)
- added U1: _Microchip_Tech_CAP1188_1_CP_TR, lcsc:QFN-24_L4.0-W4.0-P0.50-BL-EP2.5, F.Cu at (0.00, 0.00)

Commit message: Don't update PCB files
Parts:
- removed C1: 100nF ±10% 50V X7R, lcsc:C0603
- removed R1, R2, R3: 10kΩ ±1% 62.5mW, lcsc:R0402
- removed R4, R5: 1kΩ ±1% 100mW, lcsc:R0603
- removed U1: _Microchip_Tech_CAP1188_1_CP_TR, lcsc:QFN-24_L4.0-W4.0-P0.50-BL-EP2.5
