File: elec/layout/nfc/nfc.kicad_pcb (KiCad board)
At the start: 2 copper layers, 27 parts, among them U1 _NXP_Semicon_PN5321A3HN_C106_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

Commit message: Reset nfc layout
Parts:
- C1, C2: value 20pF ±5% 50V C0G -> 100nF ±10% 16V X7R; footprint lcsc:C0402 -> atopile:C0402-b3ef17
- C10, C11: value 100nF ±10% 16V X7R -> 100nF ±10% 50V X7R; footprint lcsc:C0402 -> atopile:C0603-bd72f6
- C12, C13, C17, C5, C6, C9: footprint lcsc:C0402 -> atopile:C0402-b3ef17
- C14: value 20pF ±5% 50V C0G -> 220pF ±10% 50V X7R; footprint lcsc:C0402 -> atopile:C0402-b3ef17
- C15: value 100pF ±5% 50V C0G -> 22pF ±5% 50V C0G; footprint lcsc:C0402 -> atopile:C0402-b3ef17
- C16: value 20pF ±5% 50V C0G -> 100pF ±5% 50V C0G; footprint lcsc:C0402 -> atopile:C0402-b3ef17
- C18: value 220pF ±10% 50V X7R -> 22pF ±5% 50V C0G; footprint lcsc:C0402 -> atopile:C0402-b3ef17
- C3, C7: value 100nF ±10% 16V X7R -> 10µF ±10% 10V X5R; footprint lcsc:C0402 -> atopile:C0603-bd72f6
- C4, C8: value 10µF ±10% 10V X5R -> 100nF ±10% 16V X7R; footprint lcsc:C0603 -> atopile:C0402-b3ef17
- L1, L2: value 560nH ±5% 450mA 480mΩ -> (none); footprint lcsc:IND-SMD_L1.6-W0.8-1 -> atopile:IND-SMD_L1.6-W0.8-1-cea827
- R1, R2, R3, R5: value 5.1kΩ ±1% 62.5mW -> 10kΩ ±1% 100mW; footprint lcsc:R0402 -> atopile:R0603-ebcab9
- R4: footprint lcsc:R0402 -> atopile:R0402-56259e
- U1: value _NXP_Semicon_PN5321A3HN_C106_51 -> (none); footprint lcsc:QFN-40_L6.0-W6.0-P0.50-BL-EP4.1 -> atopile:QFN-40_L6.0-W6.0-P0.50-BL-EP4.1-54a13c
- XTAL1: value Crystal -> (none); footprint lcsc:CRYSTAL-SMD_4P-L3.2-W2.5-BL -> atopile:CRYSTAL-SMD_4P-L3.2-W2.5-BL-e199c8
- moved C18 262.3 mm to (0.00, -130.0), turned to 0 degrees
- moved U1 258.1 mm to (0.00, -120.0), turned to 0 degrees
- moved R5 250.0 mm to (0.00, -110.0), turned to 0 degrees
- moved L2 237.8 mm to (0.00, -100.0), turned to 0 degrees
- moved C16 227.4 mm to (0.00, -90.0), turned to 0 degrees
- moved R2 221.4 mm to (0.00, -70.0)
- moved C12 207.3 mm to (0.00, -60.0)
- moved C15 195.9 mm to (0.00, -50.0), turned to 0 degrees
- moved L1 191.1 mm to (0.00, -40.0), turned to 0 degrees
- moved R4 187.9 mm to (0.00, -30.0)
- moved C11 176.2 mm to (3.05, 0.25), turned to 270 degrees
- moved C14 175.1 mm to (0.00, -20.0), turned to 0 degrees
- moved C10 170.1 mm to (-3.05, -0.25)
- moved C13 167.0 mm to (0.00, -10.0), turned to 0 degrees
- moved C17 163.9 mm to (0.00, 0.00), turned to 0 degrees
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Connections:
- net aux1 renamed AUX1
- net aux2 renamed AUX2
- net loadmod renamed LOADMOD
- net miso_p71 renamed MISO_P71
- net net-2 renamed TX1
- net net-4 renamed RX
- net net-8 renamed TX2
- net p30_uart_rx renamed P30_UART_RX
- net p31_uart_tx renamed P31_UART_TX
- net p32_int0 renamed P32_INT0
- net p33_int1 renamed P33_INT1
- net p34_sic_clk renamed P34_SIC_CLK
- net p70_irq renamed P70_IRQ
- net rstpd_n renamed RSTPD_N
- net sck_p72 renamed SCK_P72
- net sigin renamed SIGIN
- net signal renamed RSTOUT_N
- net sigout renamed SIGOUT
- C1 pad 1: oscillator-net -> hv
- C1 pad 2: net-1 -> gnd-1
- C10 pad 1: net-6 -> oscillator-net
- C10 pad 2: net-1 -> gnd-1
- C11 pad 1: net-1 -> OSCIN
- C11 pad 2: power_vmid-lv -> gnd-1
- C12 pad 2: net-3 -> net
- C13 pad 1: net -> line-1
- C13 pad 2: net-1 -> gnd-1
- C14 pad 2: net -> gnd-1
- C15 pad 1: net-12 -> tx_1_mid
- C15 pad 2: net-1 -> line-1
- C16 pad 1: tx_2_mid -> line
- C16 pad 2: net-12 -> gnd-1
- C17 pad 1: tx_1_mid -> tx_2_mid
- C17 pad 2: net-1 -> gnd-1
- C18 pad 2: net-1 -> line
- C2 pad 1: net-9 -> hv
- C2 pad 2: net-1 -> gnd-1
- C3 pad 1: net-6 -> hv
- C3 pad 2: net-1 -> gnd-1
- C4 pad 1: net-6 -> hv
- C4 pad 2: net-1 -> gnd-1
- C5 pad 1: net-6 -> SVDD
- C5 pad 2: net-1 -> gnd-1
- C6 pad 1: net-6 -> hv
- C6 pad 2: net-1 -> gnd-1
- C7 pad 1: net-5 -> hv
- C7 pad 2: power_svdd-lv -> gnd-1
- C8 pad 1: net-6 -> hv
- C8 pad 2: net-1 -> gnd-1
- C9 pad 1: net-6 -> gnd-1
- C9 pad 2: net-1 -> gnd
- R1 pad 1: net-10 -> oscillator-net
- R1 pad 2: hv -> OSCOUT
- R2 pad 1: net-7 -> MOSI_SDA_HSU_TX
- R2 pad 2: hv -> hv-1
- R3 pad 1: oscillator-net -> NSS_P50_SCL_HSU_RX
- R3 pad 2: net-11 -> hv-1
- R4 pad 1: net-3 -> net
- R5 pad 1: net-1 -> gnd-1
- U1 pad 1: net-1 -> gnd-1
- U1 pad 11: net-1 -> gnd-1
- U1 pad 14: net-9 -> OSCIN
- U1 pad 15: net-11 -> OSCOUT
- U1 pad 16: net-6 -> hv
- U1 pad 17: net-1 -> gnd-1
- U1 pad 18: net-1 -> gnd-1
- U1 pad 19: p35 -> nfc_ic-net
- U1 pad 20: nfc_ic-net -> nfc_ic.footprint.pins[12].net-net
- U1 pad 21: nfc_ic-net -> nfc_ic.footprint.pins[13].net-net
- U1 pad 22: nfc_ic-net -> nfc_ic.footprint.pins[14].net-net
- U1 pad 23: net-6 -> hv
- U1 pad 27: net-7 -> NSS_P50_SCL_HSU_RX
- U1 pad 28: net-10 -> MOSI_SDA_HSU_TX
- U1 pad 3: net-1 -> gnd-1
- U1 pad 37: net-5 -> SVDD
- U1 pad 39: net-6 -> hv
- U1 pad 40: net-6 -> hv
- U1 pad 41: net-1 -> gnd-1
- U1 pad 5: net-6 -> hv
- U1 pad 7: net-1 -> gnd-1
- U1 pad 8: net-6 -> hv
- U1 pad 9: net-1 -> gnd-1
- XTAL1 pad 2: net-1 -> gnd-1
- XTAL1 pad 3: net-9 -> OSCIN
- XTAL1 pad 4: net-1 -> gnd-1
Routing:
- net OSCIN: track 0.00 -> 102.7 mm
- net oscillator-net: track 5.21 -> 106.2 mm
- net net-1: track 25.8 -> 0.00 mm, vias 1 -> 0
- net net-6: track 12.3 -> 0.00 mm, vias 3 -> 0
- net net-9: track 10.3 -> 0.00 mm
- net TX1: track 8.00 -> 0.00 mm
- net net-10: track 4.67 -> 0.00 mm
- net TX2: track 3.91 -> 0.00 mm
- net tx_2_mid: track 3.78 -> 0.00 mm
- net net-7: track 3.66 -> 0.00 mm
- net RX: track 2.75 -> 0.00 mm
- net tx_1_mid: track 2.42 -> 0.00 mm
- net net-3: track 1.57 -> 0.00 mm
- net net-11: track 1.49 -> 0.00 mm
- net net: track 1.20 -> 0.00 mm
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