File: elec/layout/default/nonos.kicad_pcb (KiCad board)
At the start: 4 copper layers, 45 x 122 mm, 74 parts, among them CN1 HRSHirose_DF40C_100DS_0_4V51, CN2 HRSHirose_DF40C_100DS_0_4V51, Q1 MOSFET, U1 STUSB4500QTR, U2 _Texas_Instruments_SN74LVC1G0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, U3 _Texas_Instruments_TAS5825MRH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, U4 _HCTL_HC_TYPE_C_24P_VS9_3_5A_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, U5 JST_Sales_America_B02B_XASK_1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, U6 JST_Sales_America_B02B_XASK_1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, U7 _Texas_Instruments_TPS56637RP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

Commit message: update layout
Parts:
- removed HDR1, HDR2: HCTL_PZ254_2_04_S, lcsc:HDR-SMD_8P-P2.54-V-M-R2-C4-LS7.4
- added C31: 22µF ±20% 25V X5R, atopile:C0805-3b2e55, F.Cu at (140.0, -120.0)
- added C32: 22µF ±20% 25V X5R, atopile:C0805-3b2e55, F.Cu at (140.0, -130.0)
- added C33: 22µF ±20% 25V X5R, atopile:C0805-3b2e55, F.Cu at (140.0, -10.0)
- added D6: , atopile:SMB_L4.6-W3.6-LS5.3-RD-330cb3, F.Cu at (140.0, -70.0)
- added SW1: , atopile:SW-SMD_L6.0-W3.3-LS8.0-cfbaed, F.Cu at (50.0, 0.00)
- added SW2: , atopile:SW-SMD_L6.0-W3.3-LS8.0-cfbaed, F.Cu at (90.0, 0.00)
- added U10: , lib:HDR-SMD_8P-P2.54-V-M-R2-C4-LS7.4, F.Cu at (30.0, 0.00)
- added U11: 1kΩ ±1% 62.5mW, atopile:R0402-56259e, F.Cu at (30.0, -10.0)
- added U12: 1kΩ ±1% 62.5mW, atopile:R0402-56259e, F.Cu at (30.0, -30.0)
- added U13: 1kΩ ±1% 62.5mW, atopile:R0402-56259e, F.Cu at (30.0, -20.0)
- added U14: 1kΩ ±1% 62.5mW, atopile:R0402-56259e, F.Cu at (30.0, -40.0)
- added U15: , lib:HDR-SMD_8P-P2.54-V-M-R2-C4-LS7.4, F.Cu at (100.0, 0.00)
- added U16: 1kΩ ±1% 62.5mW, atopile:R0402-56259e, F.Cu at (100.0, -10.0)
- added U17: 1kΩ ±1% 62.5mW, atopile:R0402-56259e, F.Cu at (100.0, -30.0)
- added U18: 1kΩ ±1% 62.5mW, atopile:R0402-56259e, F.Cu at (100.0, -20.0)
- added U19: 1kΩ ±1% 62.5mW, atopile:R0402-56259e, F.Cu at (100.0, -40.0)
- added U20: , lib:HDR-SMD_8P-P2.54-V-M-R2-C4-LS7.4, F.Cu at (110.0, 0.00)
- added U21: 1kΩ ±1% 62.5mW, atopile:R0402-56259e, F.Cu at (110.0, -10.0)
- added U22: 1kΩ ±1% 62.5mW, atopile:R0402-56259e, F.Cu at (110.0, -30.0)
- added U23: 1kΩ ±1% 62.5mW, atopile:R0402-56259e, F.Cu at (110.0, -20.0)
- added U24: 1kΩ ±1% 62.5mW, atopile:R0402-56259e, F.Cu at (110.0, -40.0)
- added U25: , atopile:QFN-24_L4.0-W4.0-P0.50-BL-EP2.8-2a85a7, F.Cu at (130.0, -70.0)
- added U26: , atopile:SOIC-8_L5.0-W4.0-P1.27-LS6.0-BL-EP2.0-748c0f, F.Cu at (140.0, -80.0)
- added U8: , atopile:SMD_BD5.6-D4.1-12eb58, F.Cu at (40.0, -20.0)
- added U9: , atopile:SMD_BD5.6-D4.1-12eb58, F.Cu at (40.0, -30.0)
- added USB1: , atopile:USB-C-SMD_TYC-324G-a50b79, F.Cu at (120.0, 0.00)
- C1: value 4.7µF ±10% 35V X5R -> 4.7µF ±10% 10V X5R; footprint lcsc:C0603 -> atopile:C0603-bd72f6
- C10, C13, C14, C9: footprint lcsc:C0805 -> atopile:C0805-3b2e55
- C11, C12, C7, C8: footprint lcsc:C0603 -> atopile:C0603-bd72f6
- C15: value 4.7µF ±10% 16V X5R -> 22µF ±20% 25V X5R; footprint lcsc:C0603 -> atopile:C0805-3b2e55
- C16, C22, C23, C5, C6: footprint lcsc:C0402 -> atopile:C0402-b3ef17
- C17, C18: value 22µF ±20% 25V X5R -> 100nF ±10% 16V X7R; footprint lcsc:C0805 -> atopile:C0402-b3ef17
- C19: value 22µF ±20% 25V X5R -> 4.7µF ±10% 35V X5R; footprint lcsc:C0805 -> atopile:C0603-bd72f6
- C2: value 1µF ±10% 25V X5R -> 100nF ±10% 16V X7R; footprint lcsc:C0402 -> atopile:C0402-b3ef17
- C20, C21: value 100nF ±10% 16V X7R -> 1µF ±10% 25V X5R; footprint lcsc:C0402 -> atopile:C0402-b3ef17
- C24: value 4.7µF ±10% 25V X5R -> 100nF ±10% 50V X7R; footprint lcsc:C0805 -> atopile:C0402-b3ef17
- C25: value 4.7µF ±10% 25V X5R -> 4.7nF ±5% 50V C0G; footprint lcsc:C0805 -> atopile:C0402-b3ef17
- C26: value 4.7µF ±10% 25V X5R -> 8.2pF ±5% 50V C0G; footprint lcsc:C0805 -> atopile:C0402-b3ef17
- C27, C29: value 100nF ±10% 16V X7R -> 10µF ±10% 50V X5R; footprint lcsc:C0402 -> atopile:C0805-3b2e55
- C28: value 47µF ±20% 6.3V X5R -> 10µF ±10% 50V X5R; footprint lcsc:C0805 -> atopile:C0805-3b2e55
- C3: value 1µF ±10% 25V X5R -> 22µF ±20% 25V X5R; footprint lcsc:C0402 -> atopile:C0805-3b2e55
- C30: value 100pF ±5% 50V C0G -> 22µF ±20% 25V X5R; footprint lcsc:C0402 -> atopile:C0805-3b2e55
- C4: value 100nF ±10% 16V X7R -> 22µF ±20% 25V X5R; footprint lcsc:C0402 -> atopile:C0805-3b2e55
- CN1, CN2: value HRSHirose_DF40C_100DS_0_4V51 -> (none); footprint lcsc:CONN-SMD_DF40C-100DS-0.4V-51 -> atopile:CONN-SMD_DF40C-100DS-0.4V-51-ceffa9
- D1: value ESDA25W -> (none); footprint lcsc:SOT-323-3_L2.1-W1.3-P1.32-LS2.1-BR -> atopile:LED0603-RD-YELLOW-5af84a
- D2: footprint lcsc:DFN1610-2_L1.6-W1.0-P1.05-RD -> atopile:LED0603-RD-c81ffb
- D3: footprint lcsc:DFN1610-2_L1.6-W1.0-P1.05-RD -> atopile:SOT-323-3_L2.1-W1.3-P1.32-LS2.1-BR-ee9edb
- D4, D5: footprint lcsc:LED0805-R-RD -> atopile:DFN1610-2_L1.6-W1.0-P1.05-RD-57a24e
- FPC1: value TE_Connectivity_1_2328702_0 -> (none); footprint lcsc:FPC-SMD_10P-P0.50_HDGC_0.5K-HX-10PWB -> atopile:FPC-SMD_10P-P0.50_HDGC_0.5K-HX-10PWB-40cf1c
- L1, L2, L3, L4: value 10µH ±20% 4.5A 68mΩ -> (none); footprint lcsc:IND-SMD_L7.3-W6.8 -> atopile:IND-SMD_L7.3-W6.8-0bbdba
- L5: value 3.3µH ±20% 4A 73mΩ -> (none); footprint lcsc:IND-SMD_L4.0-W4.0 -> atopile:IND-SMD_L8.0-W8.0_SWPA8040S-2a70f8
- Q1: value MOSFET -> (none); footprint lcsc:PDFN3333-8_L3.1-W3.2-P0.65-LS3.4-BL -> atopile:PDFN3333-8_L3.1-W3.2-P0.65-LS3.4-BL-33e04e
- R1, R4: value 1kΩ ±1% 62.5mW -> 10kΩ ±1% 62.5mW; footprint lcsc:R0402 -> atopile:R0402-56259e
- R10: value 10Ω ±1% 62.5mW -> 0Ω 62.5mW; footprint lcsc:R0402 -> atopile:R0402-56259e
- R11, R12: value 10kΩ ±1% 62.5mW -> 4.7kΩ ±1% 62.5mW; footprint lcsc:R0402 -> atopile:R0402-56259e
- R13: value 10kΩ ±1% 62.5mW -> 1kΩ ±1% 62.5mW; footprint lcsc:R0402 -> atopile:R0402-56259e
- R14: value 10kΩ ±1% 62.5mW -> 100kΩ ±1% 62.5mW; footprint lcsc:R0402 -> atopile:R0402-56259e
- R15: footprint lcsc:R0402 -> atopile:R0402-56259e
- R16: value 8.2kΩ ±1% 62.5mW -> 100Ω ±1% 62.5mW; footprint lcsc:R0402 -> atopile:R0402-56259e
- R17: value 68kΩ ±1% 62.5mW -> 23.7kΩ ±1% 62.5mW; footprint lcsc:R0402 -> atopile:R0402-56259e
- R18: value 100kΩ ±1% 62.5mW -> 10kΩ ±1% 62.5mW; footprint lcsc:R0402 -> atopile:R0402-56259e
- R19: value 5.1kΩ ±1% 62.5mW -> 100kΩ ±1% 62.5mW; footprint lcsc:R0402 -> atopile:R0402-56259e
- R2, R3: value 4.7kΩ ±1% 62.5mW -> 10kΩ ±1% 62.5mW; footprint lcsc:R0402 -> atopile:R0402-56259e
- R20: value 5.1kΩ ±1% 62.5mW -> 162kΩ ±1% 62.5mW; footprint lcsc:R0402 -> atopile:R0402-56259e
- R5: value 100kΩ ±1% 62.5mW -> 2kΩ ±1% 62.5mW; footprint lcsc:R0402 -> atopile:R0402-56259e
- R6: value 22kΩ ±1% 62.5mW -> 2kΩ ±1% 62.5mW; footprint lcsc:R0402 -> atopile:R0402-56259e
- R7: value 100Ω ±1% 62.5mW -> 470Ω ±1% 100mW; footprint lcsc:R0402 -> atopile:R0603-ebcab9
- R8: value 470Ω ±1% 62.5mW -> 470Ω ±1% 100mW; footprint lcsc:R0402 -> atopile:R0603-ebcab9
- R9: value 470Ω ±1% 62.5mW -> 1kΩ ±1% 62.5mW; footprint lcsc:R0402 -> atopile:R0402-56259e
- RJ1: value _HANRUNZhongshan_HanRun_Elec_HR911130A -> (none); footprint lcsc:RJ45-TH_HR911130A -> atopile:RJ45-TH_HR911130A-5845d4
- U1: value STUSB4500QTR -> (none); footprint lcsc:QFN-24_L4.0-W4.0-P0.50-BL-EP2.8 -> atopile:SOT-23-5_L3.0-W1.7-P0.95-LS2.8-BR-9d80aa
- U2: value _Texas_Instruments_SN74LVC1G07DBVR -> (none); footprint lcsc:SOT-23-5_L3.0-W1.7-P0.95-LS2.8-BR -> atopile:SMD_BD5.6-D4.1-12eb58
- U3: value _Texas_Instruments_TAS5825MRHBR -> (none); footprint lcsc:VQFN-32_L5.0-W5.0-P0.50-TL-EP -> atopile:VQFN-32_L5.0-W5.0-P0.50-TL-EP-7b5304
- U4: value _HCTL_HC_TYPE_C_24P_VS9_3_5A_F1_1_04 -> (none); footprint lcsc:USB-C-SMD_HC-TYPE-C-24P-VS9.3-5A-F1.1-04 -> atopile:USB-C-SMD_HC-TYPE-C-24P-VS9.3-5A-F1.1-04-81dd06
- U5, U6: value JST_Sales_America_B02B_XASK_1_ALFSN -> (none); footprint lcsc:CONN-TH_B02B-XASK-1-A-LF-SN -> atopile:CONN-TH_B02B-XASK-1-A-LF-SN-8344ff
- U7: value _Texas_Instruments_TPS56637RPAR -> (none); footprint lcsc:VQFN-HR-10_L3.0-W3.0_RPA -> atopile:SMD_BD5.6-D4.1-12eb58
- moved R15 271.9 mm to (130.0, -140.0), turned to 0 degrees
- moved C28 238.0 mm to (140.0, -110.0), turned to 0 degrees
- moved C27 235.9 mm to (140.0, -100.0)
- moved R4 225.1 mm to (0.00, -30.0), turned to 0 degrees
- moved L5 218.5 mm to (140.0, -90.0), turned to 0 degrees
- moved C22 212.1 mm to (130.0, -150.0), turned to 0 degrees
- moved C4 211.7 mm to (20.0, -30.0)
- moved R2 210.0 mm to (0.00, -20.0), turned to 0 degrees
- moved R6 207.2 mm to (60.0, -50.0)
- moved R20 204.2 mm to (140.0, -140.0)
- moved R1 203.7 mm to (0.00, -10.0)
- moved C2 202.7 mm to (10.0, -10.0), turned to 0 degrees
- moved R9 198.1 mm to (130.0, -40.0), turned to 0 degrees
- moved C1 196.2 mm to (10.0, 0.00), turned to 0 degrees
- moved R3 194.7 mm to (0.00, 0.00), turned to 0 degrees
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Connections:
- net ETH_P0_N renamed cm5-pins[9]
- net ETH_P0_P renamed MDI0plus
- net ETH_P1_N renamed cm5-pins[5]
- net ETH_P1_P renamed MDI1plus
- net ETH_P2_N renamed cm5-pins[8]
- net ETH_P2_P renamed cm5-pins[10]
- net ETH_P3_N renamed MDI3_
- net ETH_P3_P renamed cm5-pins[2]-1
- net HDMI0_CK_N renamed pins[89]
- net HDMI0_CK_P renamed cm5.cm5-pins[87]-1
- net HDMI0_D0_N renamed pins[83]
- net HDMI0_D0_P renamed cm5.cm5-pins[81]
- net HDMI0_D1_N renamed pins[77]
- net HDMI0_D1_P renamed cm5.cm5-pins[75]
- net HDMI0_D2_N renamed cm5.cm5-pins[71]
- net HDMI0_D2_P renamed cm5.cm5-pins[69]
- net HDMI0_HOTPLUG renamed pins[52]
- net HDMI1_CEC renamed pins[48]
- net HDMI1_CK_N renamed pins[65]
- net HDMI1_CK_P renamed cm5.cm5-pins[63]
- net HDMI1_D0_N renamed pins[59]
- net HDMI1_D0_P renamed cm5.cm5-pins[57]
- net HDMI1_D1_N renamed cm5.cm5-pins[53]
- net HDMI1_D1_P renamed pins[51]
- net HDMI1_D2_N renamed cm5.cm5-pins[47]-1
- net HDMI1_D2_P renamed cm5.cm5-pins[45]
- net HDMI1_HOTPLUG renamed pins[42]
- net I2S_SCK renamed SCLK
- net I2S_SD renamed SDIN
- net I2S_WS renamed LRCLK
- net USB2_D_N renamed cm5-pins[2]
- net USB2_D_P renamed pins[4]
- net VCC_1V8 renamed cm5.cm5-pins[87]
- net amplifier-net renamed OUT_Bplus
- net amplifier-net-1 renamed GVDD
- net amplifier-net-10 renamed AVDD
- net amplifier-net-11 renamed BST_A_
- net amplifier-net-2 renamed OUT_B_
- net amplifier-net-3 renamed BST_B_
- net amplifier-net-4 renamed BST_Aplus
- net amplifier-net-5 renamed OUT_Aplus
- net amplifier-net-6 renamed VR_DIG
- net amplifier-net-7 renamed BST_Bplus
- net amplifier-net-8 renamed OUT_A_
- net amplifier-net-9 renamed ADR
- net net-2 renamed line-10
- net net-3 renamed line-9
- net p10 renamed cm5.rj45.connector-net
- net pd_controller.pd_controller-signal-1 renamed N_C_
- net pins[10] renamed cm5.cm5.hdi_b-pins[10]
- net pins[14] renamed cm5.cm5.hdi_b-pins[14]
- net pins[16] renamed cm5.cm5.hdi_b-pins[16]
- net pins[20] renamed cm5.cm5.hdi_b-pins[20]
- net pins[23] renamed cm5.cm5.hdi_b-pins[23]
- net pins[26] renamed cm5.cm5.hdi_b-pins[26]
- net pins[27] renamed cm5.cm5.hdi_b-pins[27]
- net pins[28] renamed cm5.cm5.hdi_b-pins[28]
- net pins[45] renamed cm5-pins[45]
- net pins[5] renamed cm5.cm5.hdi_b-pins[5]
- net pins[63] renamed cm5.cm5.hdi_a-pins[63]
- net pins[69] renamed cm5.cm5.hdi_a-pins[69]
- net pins[71] renamed cm5.cm5.hdi_a-pins[71]
- net pins[75] renamed cm5.cm5.hdi_a-pins[75]
- net pins[8] renamed cm5.cm5.hdi_b-pins[8]
- net pins[95] renamed cm5.cm5.hdi_b-pins[95]
- net pins[9] renamed cm5.cm5.hdi_b-pins[9]
- net processor-pins[40] renamed cm5.cm5-pins[40]
- net processor-pins[44] renamed cm5.cm5-pins[44]-1
- net processor-pins[44]-1 renamed cm5.cm5-pins[44]
- net processor-pins[46] renamed cm5-pins[46]
- net processor-pins[46]-1 renamed cm5.cm5-pins[46]
- net processor-pins[49] renamed cm5-pins[49]
- net processor-pins[98] renamed cm5.cm5-pins[98]
- net processor-pins[99] renamed cm5.cm5-pins[99]
- net processor-signal renamed cm5.cm5-pins[23]
- net processor-signal-2 renamed cm5.cm5-pins[47]
- net processor-signal-4 renamed cm5-pins[26]
- net processor-signal-5 renamed cm5-pins[28]
- net processor-signal-6 renamed pins[30]
- net processor.hdi_a-pins[15] renamed cm5.cm5.hdi_a-pins[15]
- net processor.hdi_a-pins[17] renamed cm5.cm5.hdi_a-pins[17]
- net processor.hdi_a-pins[56] renamed cm5.cm5.hdi_a-pins[56]
- net processor.hdi_a-pins[62] renamed cm5.cm5.hdi_a-pins[62]
- net processor.hdi_a-pins[68] renamed cm5.cm5.hdi_a-pins[68]
- net processor.hdi_a-pins[74] renamed cm5.cm5.hdi_a-pins[74]
- net processor.hdi_a-pins[88] renamed cm5.cm5.hdi_a-pins[88]
- net processor.hdi_a-pins[93] renamed cm5.cm5.hdi_a-pins[93]
- net processor.hdi_a-pins[98] renamed cm5.cm5.hdi_a-pins[98]
- net processor.hdi_a-pins[99] renamed cm5.cm5.hdi_a-pins[99]
- net processor.hdi_b-pins[15] renamed cm5.cm5.hdi_b-pins[15]
- net processor.hdi_b-pins[17] renamed cm5.cm5.hdi_b-pins[17]
- net processor.hdi_b-pins[34] renamed pins[34]
- net processor.hdi_b-pins[35] renamed pins[35]
- net processor.hdi_b-pins[39] renamed pins[39]
- net processor.hdi_b-pins[40] renamed cm5.cm5.hdi_b-pins[40]
- net processor.hdi_b-pins[49] renamed cm5.cm5.hdi_b-pins[49]
- net processor.hdi_b-pins[56] renamed cm5-pins[56]
- net processor.hdi_b-pins[62] renamed cm5-pins[62]
- net processor.hdi_b-pins[68] renamed cm5-pins[68]
- net processor.hdi_b-pins[74] renamed cm5.cm5.hdi_b-pins[74]
- net processor.hdi_b-pins[88] renamed cm5.cm5.hdi_b-pins[88]
- net processor.hdi_b-pins[92] renamed cm5.cm5.hdi_b-pins[92]
- net processor.hdi_b-pins[93] renamed cm5.cm5.hdi_b-pins[93]
- net processor.hdi_b-pins[94] renamed cm5.cm5.hdi_b-pins[94]
- net rj45.connector-net renamed cm5.rj45.connector-net-1
- net sbu2 renamed usb_connector-SBU2
- net ssrxn1 renamed SSRXN1
- net ssrxn2 renamed usb_connector.connector-SSRXN2
- net ssrxp1 renamed SSRXP1
- net ssrxp2 renamed usb_connector.connector-SSRXP2
- net sstxn1 renamed SSTXN1
- net sstxn2 renamed usb_connector.connector-SSTXN2
- net sstxp1 renamed SSTXP1
- net sstxp2 renamed usb_connector.connector-SSTXP2
- net usb_connector-net renamed DP2
- net usb_connector-net-1 renamed DN2
- net usb_connector-signal renamed SBU1
- C1 pad 1: GND -> hv-1
- C1 pad 2: VBUS -> gnd
- C10 pad 2: GND -> gnd
- C13 pad 1: net-1 -> line-4
- C13 pad 2: GND -> gnd
- C14 pad 1: net -> line-7
- C14 pad 2: GND -> gnd
- C15 pad 1: VCC_3V3 -> hv-2
- C15 pad 2: GND -> gnd
- C16 pad 1: VCC_3V3 -> hv-2
- C16 pad 2: GND -> gnd
- C17 pad 1: VSINK_VCC -> hv-2
- C17 pad 2: GND -> gnd
- C18 pad 1: VSINK_VCC -> hv-2
- C18 pad 2: GND -> gnd
- C19 pad 1: VSINK_VCC -> gnd
- C19 pad 2: GND -> VBUS
- C2 pad 1: GND -> hv-1
- C2 pad 2: VREG_1V2 -> gnd
- C20 pad 1: VSINK_VCC -> gnd
- C20 pad 2: GND -> pd_controller.pd_controller-hv
- C21 pad 1: VSINK_VCC -> gnd
- C21 pad 2: GND -> pd_controller.pd_controller-hv-1
- C22 pad 1: VSINK_VCC -> pd_controller.pd_controller-net
- C22 pad 2: GND -> VBUS
- C23 pad 2: GND -> gnd
- C24 pad 1: VSINK_VCC -> BOOT
- C24 pad 2: GND -> SW
- C25 pad 1: VSINK_VCC -> regulator_5v-net
- C25 pad 2: GND -> gnd
- C26 pad 1: VSINK_VCC -> COMP
- C26 pad 2: GND -> gnd
- C27 pad 1: VSINK_VCC -> hv-2
- C27 pad 2: GND -> gnd
- C28 pad 1: VCC_5V -> hv-2
- C28 pad 2: GND -> gnd
- C29 pad 1: regulator-net -> hv-2
- C29 pad 2: regulator-net-1 -> gnd
- C3 pad 1: GND -> hv-2
- C3 pad 2: VREG_2V7 -> gnd
- C30 pad 1: regulator-net-2 -> hv
- C30 pad 2: regulator-net-3 -> gnd
- C4 pad 1: pd_controller-net-3 -> hv-2
- C4 pad 2: VBUS -> gnd
- C5 pad 2: GND -> gnd
- C6 pad 2: GND -> gnd
- C9 pad 2: GND -> gnd
- CN1 pad 1: GND -> gnd
- CN1 pad 10: processor-net-2 -> pins[19]
- CN1 pad 100: GND -> gnd
- CN1 pad 11: GND -> gnd
- CN1 pad 14: UART_TX -> cm5-pins[27]
- CN1 pad 15: signal-3 -> PDNh
- CN1 pad 16: GND -> gnd
- CN1 pad 17: signal-4 -> pins[33]
- CN1 pad 18: processor.hdi_a-pins[35] -> line-6
- CN1 pad 20: processor-pins[39] -> line-11
- CN1 pad 21: GND -> gnd
- CN1 pad 22: processor-signal-3 -> line-1
- CN1 pad 26: GND -> gnd
- CN1 pad 27: signal-5 -> pins[53]
- CN1 pad 28: signal-2 -> line-2
- CN1 pad 29: signal-1 -> cm5-pins[57]
- CN1 pad 30: GND -> gnd
- CN1 pad 33: GND -> gnd
- CN1 pad 37: GND -> gnd
- CN1 pad 39: VCC_3V3 -> hv-1
- CN1 pad 4: GND -> gnd
- CN1 pad 40: SCL -> pins[79]
- CN1 pad 41: SDA -> cm5.cm5.hdi_a-pins[81]
- CN1 pad 42: VCC_3V3 -> hv-1
- CN1 pad 43: VCC_3V3 -> hv-1
- CN1 pad 48: PWR_LED -> cm5.cm5.hdi_a-pins[95]
- CN1 pad 49: GND -> gnd
- CN1 pad 53: processor.hdi_a-pins[94] -> cm5.cm5-pins[94]
- CN1 pad 54: processor.hdi_a-pins[92] -> cm5-pins[92]
- CN1 pad 57: VCC_5V -> hv
- CN1 pad 58: VCC_5V -> hv
- CN1 pad 59: VCC_5V -> hv
- CN1 pad 60: VCC_5V -> hv
- CN1 pad 61: VCC_5V -> hv
- CN1 pad 62: VCC_5V -> hv
- CN1 pad 65: GND -> gnd
- CN1 pad 68: GND -> gnd
- CN1 pad 7: GND -> gnd
- CN1 pad 71: GND -> gnd
- CN1 pad 73: UART_RX -> line-5
- CN1 pad 74: GND -> gnd
- CN1 pad 75: pins[50] -> line-12
- CN1 pad 79: GND -> gnd
- CN1 pad 81: processor-signal-1 -> line
- CN1 pad 82: signal -> line-8
- CN1 pad 83: processor.hdi_a-pins[34] -> line-3
- CN1 pad 84: GND -> gnd
- CN1 pad 89: GND -> gnd
- CN1 pad 90: GND -> cm5.cm5-pins[20]
- CN1 pad 92: ETH_LED_ACTIVITY -> cm5-pins[16]
- CN1 pad 93: ETH_LED_LINK -> cm5-pins[14]
- CN1 pad 94: GND -> gnd
- CN1 pad 97: GND -> gnd
- CN2 pad 10: GND -> gnd
- CN2 pad 13: GND -> gnd
- CN2 pad 16: GND -> gnd
- CN2 pad 17: pins[33] -> cm5-pins[33]
- CN2 pad 19: GND -> gnd
- CN2 pad 22: GND -> gnd
- CN2 pad 28: GND -> gnd
- CN2 pad 31: GND -> gnd
- CN2 pad 34: GND -> gnd
- CN2 pad 37: GND -> gnd
- CN2 pad 4: GND -> gnd
- CN2 pad 40: GND -> gnd
- CN2 pad 43: GND -> gnd
- CN2 pad 46: GND -> gnd
- CN2 pad 49: GND -> gnd
- CN2 pad 52: GND -> gnd
- CN2 pad 55: GND -> gnd
- CN2 pad 58: GND -> gnd
- CN2 pad 61: GND -> gnd
- CN2 pad 64: GND -> gnd
- CN2 pad 67: GND -> gnd
- CN2 pad 7: GND -> gnd
- CN2 pad 70: GND -> gnd
- CN2 pad 73: GND -> gnd
- CN2 pad 75: HDMI0_CEC -> pins[50]
- CN2 pad 82: GND -> gnd
- CN2 pad 85: GND -> gnd
- CN2 pad 88: GND -> gnd
- CN2 pad 91: GND -> gnd
- CN2 pad 94: GND -> gnd
- CN2 pad 97: GND -> gnd
- D1 pad 1: CC1 -> cm5.cm5-cathode-1
- D1 pad 2: CC2 -> hv-1
- D2 pad 1: VBUS -> cm5.cm5-cathode
- D2 pad 2: GND -> hv-1
- D3 pad 1: VSINK_VCC -> CC1
- D3 pad 2: GND -> CC2
- D4 pad 1: VCC_3V3 -> VBUS
- D4 pad 2: processor-net-3 -> gnd
- D5 pad 1: VCC_3V3 -> hv-2
- D5 pad 2: processor-net-1 -> gnd
- FPC1 pad 1: SDA -> line-1
- FPC1 pad 10: signal -> line-6
- FPC1 pad 11: board_to_board_connector.board_to_board_connector-net -> board_to_board_connector.board_to_board_connector-net-1
- FPC1 pad 12: board_to_board_connector.board_to_board_connector-net-1 -> board_to_board_connector.board_to_board_connector-net
- FPC1 pad 2: SCL -> line-11
- FPC1 pad 3: GND -> line
- FPC1 pad 4: VCC_5V -> line-8
- FPC1 pad 5: VCC_3V3 -> gnd
- FPC1 pad 6: GND -> hv-1
- FPC1 pad 7: signal-5 -> hv
- FPC1 pad 8: signal-4 -> gnd
- FPC1 pad 9: signal-3 -> line-3
- L3 pad 2: net-1 -> line-4
- L4 pad 2: net -> line-7
- L5 pad 1: VCC_5V -> SW
- L5 pad 2: regulator-net-1 -> hv
- Q1 pad 4: pd_controller-net-2 -> gate
- Q1 pad 5: VSINK_VCC -> hv-2
- Q1 pad 6: VSINK_VCC -> hv-2
- Q1 pad 7: VSINK_VCC -> hv-2
- Q1 pad 8: VSINK_VCC -> hv-2
- Q1 pad 9: VSINK_VCC -> hv-2
- R1 pad 1: VBUS -> pins[33]
- R1 pad 2: pd_controller-net-1 -> hv-1
- R10 pad 2: GND -> gnd
- R11 pad 1: signal-1 -> line-3
- R11 pad 2: VCC_3V3 -> hv-1
- R12 pad 1: signal-7 -> line-6
- R12 pad 2: VCC_3V3 -> hv-1
- R13 pad 1: signal-2 -> VBUS
- R13 pad 2: VCC_3V3 -> VBUS_VS_DISCH
- R14 pad 1: signal-6 -> gate
- R14 pad 2: VCC_3V3 -> hv-2
- R15 pad 1: VCC_5V -> gate
- R15 pad 2: regulator-net-2 -> VBUS_EN_SNK
- R16 pad 1: GND -> gate
- R16 pad 2: regulator-net-3 -> pd_controller.pd_controller-net
- R17 pad 1: VCC_5V -> COMP
- R17 pad 2: regulator-net-3 -> regulator_5v-net
- R18 pad 1: VCC_5V -> FB
- R18 pad 2: regulator-net-4 -> gnd
- R19 pad 1: processor-net-3 -> hv
- R19 pad 2: processor-net-2 -> FB
- R2 pad 1: SCL -> line-2
- R2 pad 2: VCC_3V3 -> hv-1
- R20 pad 1: processor-net-1 -> RT_CLK
- R20 pad 2: processor-net -> gnd
- R3 pad 1: SDA -> PDNh
- R3 pad 2: VCC_3V3 -> hv-1
- R4 pad 1: VBUS -> pins[53]
- R4 pad 2: pd_controller-net -> hv-1
- R5 pad 1: pd_controller-net-2 -> cm5.cm5-cathode-1
- R5 pad 2: VSINK_VCC -> cm5.cm5-pins[20]
- R6 pad 1: pd_controller-net-2 -> cm5.cm5-cathode
- R6 pad 2: pd_controller-net-4 -> Y
- R7 pad 1: pd_controller-net-2 -> hv-1
- R7 pad 2: pd_controller-net-3 -> cm5.rj45-anode-1
- R8 pad 1: VCC_3V3 -> hv-1
- R8 pad 2: rj45-net-1 -> cm5.rj45-anode
- R9 pad 1: VCC_3V3 -> VBUS
- R9 pad 2: rj45-net -> DISCH
- RJ1 pad 11: ETH_LED_LINK -> cm5.rj45-anode-1
- RJ1 pad 12: rj45-net-1 -> cm5-pins[14]
- RJ1 pad 13: rj45-net -> cm5-pins[16]
- RJ1 pad 14: ETH_LED_ACTIVITY -> cm5.rj45-anode
- RJ1 pad SHIELD0: GND -> gnd
- RJ1 pad SHIELD1: GND -> gnd
- U1 pad 2: CC1 -> cm5.cm5-pins[94]
- U1 pad 3: pd_controller.pd_controller.footprint.pins[18].net-net -> gnd
- U1 pad 4: CC2 -> Y
- U1 pad 5: pd_controller.pd_controller-signal -> hv-1
- U2 pad 1: n_c_ -> gnd
- U2 pad 2: PWR_LED -> gnd
- U2 pad 4: processor-net -> gnd
- U3 pad 10: signal-7 -> line-2
- U3 pad 11: signal-6 -> pins[53]
- U3 pad 15: SDA -> line-6
- U3 pad 16: SCL -> line-3
- U3 pad 17: signal-2 -> PDNh
- U3 pad 20: GND -> gnd
- U3 pad 21: VSINK_VCC -> hv-2
- U3 pad 22: VSINK_VCC -> hv-2
- U3 pad 25: GND -> gnd
- U3 pad 26: GND -> gnd
- U3 pad 3: VSINK_VCC -> hv-2
- U3 pad 31: GND -> gnd
- U3 pad 32: GND -> gnd
- U3 pad 33: GND -> gnd
- U3 pad 4: VSINK_VCC -> hv-2
- U3 pad 5: GND -> gnd
- U3 pad 6: VCC_3V3 -> hv-1
- U3 pad 9: signal-1 -> pins[33]
- U4 pad 25: GND -> gnd
- U4 pad 26: GND -> gnd
- U4 pad 27: GND -> gnd
- U4 pad 28: GND -> gnd
- U4 pad A1: GND -> gnd
- U4 pad A12: GND -> gnd
- U4 pad B1: GND -> gnd
- U4 pad B12: GND -> gnd
- U6 pad 1: net-1 -> line-7
- U6 pad 2: net -> line-4
- U7 pad 1: en -> gnd
- U7 pad 2: regulator-net-3 -> gnd
- U7 pad 3: GND -> gnd
- U7 pad 4: regulator-net-4 -> gnd
Routing:
- net (no net): track 0.00 -> 2251.3 mm, vias 0 -> 174
- net SDA: track 157.3 -> 0.00 mm, vias 6 -> 0
- net SCL: track 154.3 -> 0.00 mm, vias 6 -> 0
- net VCC_5V: track 136.7 -> 0.00 mm, vias 4 -> 0
- net signal: track 87.2 -> 0.00 mm, vias 3 -> 0
- net signal-5: track 84.9 -> 0.00 mm, vias 3 -> 0
- net signal-3: track 82.1 -> 0.00 mm, vias 3 -> 0
- net signal-4: track 82.1 -> 0.00 mm, vias 3 -> 0
- net SCLK: track 79.1 -> 0.00 mm, vias 4 -> 0
- net ETH_LED_ACTIVITY: track 78.5 -> 0.00 mm, vias 2 -> 0
- net GND: track 76.4 -> 0.00 mm, vias 45 -> 0
- net ETH_LED_LINK: track 70.0 -> 0.00 mm, vias 2 -> 0
- net MDI3_: track 69.5 -> 0.00 mm, vias 2 -> 0
- net LRCLK: track 69.4 -> 0.00 mm, vias 4 -> 0
- net cm5-pins[2]-1: track 68.8 -> 0.00 mm, vias 2 -> 0
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- added copper zone on B.Cu, net (none)
- added copper zone on F.Cu, net (none)
- added copper zone on In1.Cu, net (none)
- added copper zone on In2.Cu, net (none)
- removed copper zone on F.Cu, net GND
- removed copper zone on In2.Cu, net GND
- removed copper zone on F.Cu, net VBUS
- removed copper zone on B.Cu, net VCC_3V3
- removed copper zone on In1.Cu, net VCC_3V3
- removed copper zone on F.Cu, net VCC_5V
- removed copper zone on B.Cu, net VSINK_VCC
- removed copper zone on F.Cu, net VSINK_VCC
- removed copper zone on F.Cu, net net
- removed copper zone on F.Cu, net net-1

Commit message: layout updates
Parts:
- R19: value 100kΩ ±1% 62.5mW -> 1kΩ ±1% 62.5mW
- moved C22 284.2 mm to (161.1, 132.5)
- moved R15 277.0 mm to (159.3, 135.4), turned to -90 degrees
- moved R20 274.6 mm to (134.5, 134.5), turned to 180 degrees
- moved C32 271.6 mm to (133.6, 141.6), turned to 180 degrees
- moved C21 264.8 mm to (159.4, 133.1), turned to 90 degrees
- moved C31 258.0 mm to (133.6, 137.9), turned to 180 degrees
- moved C20 254.7 mm to (158.4, 133.1), turned to 90 degrees
- moved C28 244.2 mm to (143.0, 134.2), turned to 90 degrees
- moved R13 244.0 mm to (162.8, 131.8), turned to 90 degrees
- moved L5 238.7 mm to (137.8, 148.7)
- moved D4 235.8 mm to (165.2, 133.2), turned to -90 degrees
- moved C27 234.2 mm to (141.2, 134.2), turned to 90 degrees
- moved C19 223.5 mm to (165.2, 130.7), turned to -90 degrees
- moved U26 220.6 mm to (138.4, 140.6), turned to 180 degrees
- moved D6 211.2 mm to (143.2, 141.2), turned to 90 degrees
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Connections:
- net DP2 renamed DP1
- net MDI3_ renamed cm5-pins[4]-1
- net cm5-pins[10] renamed MDI2plus
- net cm5-pins[2] renamed pins[2]
- net cm5-pins[2]-1 renamed MDI3plus
- net cm5-pins[5] renamed MDI1_
- net cm5.cm5-pins[87] renamed cm5.cm5-pins[89]-1
- net cm5.cm5-pins[87]-1 renamed pins[87]
- net cm5.cm5.hdi_b-pins[10] renamed pins[10]
- net cm5.cm5.hdi_b-pins[5] renamed pins[5]
- net pd_controller.usb_connector-SSTXN2 renamed B3
- net pd_controller.usb_connector-SSTXP2 renamed B2
- net pins[4] renamed cm5-pins[4]
- net pins[89] renamed cm5.cm5-pins[89]
- net usb_connector.connector-SSTXN2 renamed SSTXN2
- net usb_connector.connector-SSTXP2 renamed SSTXP2
- C1 pad 1: hv-1 -> hv
- C10 pad 1: line-10 -> line-6
- C13 pad 1: line-4 -> line-11
- C14 pad 1: line-7 -> line
- C2 pad 1: hv-1 -> hv
- C30 pad 1: hv -> hv-1
- C31 pad 1: hv -> hv-1
- C32 pad 1: hv -> hv-1
- C33 pad 1: hv -> hv-1
- C9 pad 1: line-9 -> line-3
- CN1 pad 18: line-6 -> line-10
- CN1 pad 20: line-11 -> line-12
- CN1 pad 22: line-1 -> line-4
- CN1 pad 39: hv-1 -> hv
- CN1 pad 42: hv-1 -> hv
- CN1 pad 43: hv-1 -> hv
- CN1 pad 57: hv -> hv-1
- CN1 pad 58: hv -> hv-1
- CN1 pad 59: hv -> hv-1
- CN1 pad 60: hv -> hv-1
- CN1 pad 61: hv -> hv-1
- CN1 pad 62: hv -> hv-1
- CN1 pad 73: line-5 -> line-9
- CN1 pad 75: line-12 -> line-1
- CN1 pad 81: line -> line-7
- CN1 pad 83: line-3 -> line-5
- D1 pad 1: cm5.cm5-cathode-1 -> cm5.cm5-cathode
- D1 pad 2: hv-1 -> hv
- D2 pad 1: cm5.cm5-cathode -> cm5.cm5-cathode-1
- D2 pad 2: hv-1 -> hv
- FPC1 pad 1: line-1 -> line-4
- FPC1 pad 10: line-6 -> line-10
- FPC1 pad 2: line-11 -> line-12
- FPC1 pad 3: line -> line-7
- FPC1 pad 6: hv-1 -> hv
- FPC1 pad 7: hv -> hv-1
- FPC1 pad 9: line-3 -> line-5
- L1 pad 2: line-9 -> line-3
- L2 pad 2: line-10 -> line-6
- L3 pad 2: line-4 -> line-11
- L4 pad 2: line-7 -> line
- L5 pad 2: hv -> hv-1
- R1 pad 2: hv-1 -> hv
- R11 pad 1: line-3 -> line-5
- R11 pad 2: hv-1 -> hv
- R12 pad 1: line-6 -> line-10
- R12 pad 2: hv-1 -> hv
- R19 pad 1: hv -> hv-1
- R2 pad 2: hv-1 -> hv
- R3 pad 2: hv-1 -> hv
- R4 pad 2: hv-1 -> hv
- R5 pad 1: cm5.cm5-cathode-1 -> cm5.cm5-cathode
- R6 pad 1: cm5.cm5-cathode -> cm5.cm5-cathode-1
- R7 pad 1: hv-1 -> hv
- R8 pad 1: hv-1 -> hv
- U1 pad 5: hv-1 -> hv
- U25 pad 7: line-3 -> line-5
- U25 pad 8: line-6 -> line-10
- U3 pad 15: line-6 -> line-10
- U3 pad 16: line-3 -> line-5
- U3 pad 6: hv-1 -> hv
- U5 pad 1: line-10 -> line-6
- U5 pad 2: line-9 -> line-3
- U6 pad 1: line-7 -> line
- U6 pad 2: line-4 -> line-11
Routing:
- net (no net): track 2251.3 -> 22.9 mm, vias 174 -> 0
- net gnd: track 0.00 -> 84.6 mm, vias 0 -> 36
- net hv-2: track 0.00 -> 20.9 mm, vias 0 -> 7
- net line-9: track 16.7 -> 0.00 mm
- net SW: track 0.00 -> 16.2 mm
- net CC2: track 0.00 -> 13.0 mm, vias 0 -> 2
- net CC1: track 0.00 -> 12.9 mm, vias 0 -> 2
- net hv-1: track 0.00 -> 12.4 mm, vias 0 -> 8
- net line-10: track 14.9 -> 4.26 mm
- net VBUS: track 0.00 -> 9.89 mm
- net COMP: track 0.00 -> 9.00 mm
- net FB: track 0.00 -> 8.75 mm
- net line-3: track 0.00 -> 8.52 mm
- net line-6: track 0.00 -> 8.50 mm
- net line-11: track 0.00 -> 8.48 mm
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- added copper zone on F.Cu, net SW
- added copper zone on F.Cu, net VBUS
- added copper zone on B.Cu, net gnd
- added copper zone on F.Cu, net gnd
- added copper zone on F.Cu, net hv-1
- added copper zone on F.Cu, net hv-2
- added copper zone on F.Cu, net line
- added copper zone on F.Cu, net line-11
- added copper zone on F.Cu, net line-3
- added copper zone on F.Cu, net line-6
- removed copper zone on F.Cu, net line-10
- removed copper zone on F.Cu, net line-9
Other:
- board size 45 x 122 mm -> 45 x 167 mm
- board text removed: "NONOS"
