File: elec/layout/hat/hat.kicad_pcb (KiCad board)
At the start: 4 copper layers, 108 x 115.9 mm, 83 parts

Commit message: nonos building
Parts:
- removed L1, L2: , Murata_Electronics_LQW18CNR56J00D:IND-SMD_L1.6-W0.8-1
- added U27: 560nH ±5% 450mA 550mΩ, TDK_NLV32T_R56J_EF:IND-SMD_L3.2-W2.5, F.Cu at (0.00, 0.00)
- added U28: 560nH ±5% 450mA 550mΩ, TDK_NLV32T_R56J_EF:IND-SMD_L3.2-W2.5, F.Cu at (0.00, -10.0)
Connections:
- net DIN renamed -DIN-0
- net DIN-1 renamed -DIN-1
- net DOUT renamed -DOUT-0
- net DOUT-1 renamed -DOUT-1
- net DOUT-10 renamed -DOUT-10
- net DOUT-11 renamed -DOUT-11
- net DOUT-12 renamed -DOUT-12
- net DOUT-13 renamed -DOUT-13
- net DOUT-14 renamed -DOUT-14
- net DOUT-15 renamed -DOUT-15
- net DOUT-16 renamed -DOUT-16
- net DOUT-17 renamed -DOUT-17
- net DOUT-18 renamed -DOUT-18
- net DOUT-19 renamed -DOUT-19
- net DOUT-2 renamed -DOUT-2
- net DOUT-20 renamed -DOUT-20
- net DOUT-3 renamed -DOUT-3
- net DOUT-4 renamed -DOUT-4
- net DOUT-5 renamed -DOUT-5
- net DOUT-6 renamed -DOUT-6
- net DOUT-7 renamed -DOUT-7
- net DOUT-8 renamed -DOUT-8
- net DOUT-9 renamed -DOUT-9
- net hv renamed -hv-0
- net hv-1 renamed -hv-1
- net line renamed -line-0
- net line-1 renamed -line-1
- net line-2 renamed -line-2
- net line-3 renamed -line-3

Commit message: update hat layout
Parts:
- removed U27, U28: 560nH ±5% 450mA 550mΩ, TDK_NLV32T_R56J_EF:IND-SMD_L3.2-W2.5
- added L1: , Murata_Electronics_LQW18CNR56J00D:IND-SMD_L1.6-W0.8-1, F.Cu at (153.3, 55.6)
- added L2: , Murata_Electronics_LQW18CNR56J00D:IND-SMD_L1.6-W0.8-1, F.Cu at (152.0, 55.6)
- moved R6 8.24 mm to (149.1, 101.0), turned to 180 degrees
- moved R7 8.02 mm to (154.5, 106.1), turned to -90 degrees
- moved C43 0.69 mm to (153.3, 107.2)
- moved R3 0.69 mm to (149.1, 102.0)
- moved C12 0.11 mm to (150.7, 55.4)
- moved C13 0.11 mm to (153.8, 50.1)
- moved C14 0.11 mm to (153.1, 51.8)
- moved C15 0.11 mm to (151.4, 50.2)
- moved C16 0.11 mm to (152.1, 51.8)
- moved C29 0.11 mm to (157.4, 61.0)
- moved C32 0.11 mm to (146.4, 64.5)
- moved C33 0.11 mm to (146.6, 65.8)
- moved C34 0.11 mm to (155.1, 57.1)
- moved C36 0.11 mm to (151.3, 58.0)
- moved C37 0.11 mm to (151.1, 67.6)
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Connections:
- net -DIN-0 renamed B
- net -DIN-1 renamed data_out-DIN
- net -DOUT-0 renamed leds[1]-data_in-DIN
- net -DOUT-1 renamed leds[11]-data_in-DIN
- net -DOUT-10 renamed leds[20]-data_in-DIN
- net -DOUT-11 renamed leds[2]-data_in-DIN
- net -DOUT-12 renamed leds[21]-data_in-DIN
- net -DOUT-13 renamed leds[22]-data_in-DIN
- net -DOUT-14 renamed leds[3]-data_in-DIN
- net -DOUT-15 renamed leds[4]-data_in-DIN
- net -DOUT-16 renamed leds[5]-data_in-DIN
- net -DOUT-17 renamed leds[6]-data_in-DIN
- net -DOUT-18 renamed leds[7]-data_in-DIN
- net -DOUT-19 renamed leds[8]-data_in-DIN
- net -DOUT-2 renamed leds[12]-data_in-DIN
- net -DOUT-20 renamed leds[9]-data_in-DIN
- net -DOUT-3 renamed leds[13]-data_in-DIN
- net -DOUT-4 renamed leds[14]-data_in-DIN
- net -DOUT-5 renamed leds[15]-data_in-DIN
- net -DOUT-6 renamed leds[16]-data_in-DIN
- net -DOUT-7 renamed leds[17]-data_in-DIN
- net -DOUT-8 renamed leds[18]-data_in-DIN
- net -DOUT-9 renamed leds[19]-data_in-DIN
- net -hv-0 renamed power_b-VCC
- net -line-0 renamed SDA
- net -line-1 renamed SCL
- net -line-2 renamed antenna_P
- net -line-3 renamed antenna_N
- net VMID renamed power_vmid-VCC
- net input renamed OSCIN
- net leds[22]-DOUT renamed DOUT
- net nfc.package.footprint.pins[12].net-net renamed footprint-net-0
- net nfc.package.footprint.pins[13].net-net renamed footprint-net-1
- net nfc.package.footprint.pins[14].net-net renamed footprint-net-2
- net output renamed OSCOUT
- C1 pad 2: gnd -> GND
- C10 pad 2: gnd -> GND
- C11 pad 2: gnd -> GND
- C13 pad 2: gnd -> GND
- C15 pad 2: gnd -> GND
- C17 pad 2: gnd -> GND
- C18 pad 2: gnd -> GND
- C19 pad 2: gnd -> GND
- C2 pad 2: gnd -> GND
- C20 pad 2: gnd -> GND
- C21 pad 2: gnd -> GND
- C22 pad 2: gnd -> GND
- C23 pad 2: gnd -> GND
- C24 pad 2: gnd -> GND
- C25 pad 2: gnd -> GND
- C26 pad 2: gnd -> GND
- C27 pad 2: gnd -> GND
- C28 pad 2: gnd -> GND
- C29 pad 1: -hv-1 -> power-VCC
- C29 pad 2: gnd -> GND
- C3 pad 2: gnd -> GND
- C30 pad 1: -hv-1 -> power-VCC
- C30 pad 2: gnd -> GND
- C31 pad 2: gnd -> GND
- C32 pad 2: gnd -> GND
- C33 pad 1: -hv-1 -> power-VCC
- C33 pad 2: gnd -> GND
- C34 pad 1: -hv-1 -> power-VCC
- C34 pad 2: gnd -> GND
- C35 pad 1: -hv-1 -> power-VCC
- C35 pad 2: gnd -> GND
- C36 pad 1: -hv-1 -> power-VCC
- C36 pad 2: gnd -> GND
- C37 pad 1: -hv-1 -> power-VCC
- C37 pad 2: gnd -> GND
- C38 pad 1: -hv-1 -> power-VCC
- C38 pad 2: gnd -> GND
- C39 pad 1: -hv-1 -> power-VCC
- C39 pad 2: gnd -> GND
- C4 pad 2: gnd -> GND
- C40 pad 2: gnd -> GND
- C41 pad 2: gnd -> GND
- C42 pad 2: gnd -> GND
- C43 pad 1: -hv-1 -> power-VCC
- C43 pad 2: gnd -> GND
- C44 pad 1: -hv-1 -> power-VCC
- C44 pad 2: gnd -> GND
- C45 pad 2: gnd -> GND
- C5 pad 2: gnd -> GND
- C6 pad 2: gnd -> GND
- C7 pad 2: gnd -> GND
- C8 pad 2: gnd -> GND
- C9 pad 2: gnd -> GND
- FPC1 pad 4: gnd -> GND
- FPC1 pad 5: -hv-1 -> power-VCC
- FPC1 pad 6: gnd -> GND
- R1 pad 2: -hv-1 -> power-VCC
- R2 pad 2: -hv-1 -> power-VCC
- R3 pad 2: gnd -> GND
- R6 pad 1: RESET -> nALERT_nBC_IRQ
- R6 pad 2: gnd -> power-VCC
- R7 pad 1: nALERT_nBC_IRQ -> RESET
- R7 pad 2: -hv-1 -> GND
- U1 pad 2: gnd -> GND
- U10 pad 2: gnd -> GND
- U11 pad 2: gnd -> GND
- U12 pad 2: gnd -> GND
- U13 pad 2: gnd -> GND
- U14 pad 2: gnd -> GND
- U15 pad 2: gnd -> GND
- U16 pad 2: gnd -> GND
- U17 pad 2: gnd -> GND
- U18 pad 2: gnd -> GND
- U19 pad 2: gnd -> GND
- U2 pad 2: gnd -> GND
- U20 pad 2: gnd -> GND
- U21 pad 2: gnd -> GND
- U22 pad 2: gnd -> GND
- U23 pad 2: gnd -> GND
- U24 pad 2: gnd -> GND
- U25 pad 23: -hv-1 -> power-VCC
- U25 pad 25: gnd -> GND
- U26 pad 1: -hv-1 -> power-VCC
- U26 pad 2: gnd -> GND
- U26 pad 5: -hv-1 -> power-VCC
- U3 pad 2: gnd -> GND
- U4 pad 2: gnd -> GND
- U5 pad 2: gnd -> GND
- U6 pad 2: gnd -> GND
- U7 pad 1: gnd -> GND
- U7 pad 11: gnd -> GND
- U7 pad 16: -hv-1 -> power-VCC
- U7 pad 17: gnd -> GND
- U7 pad 18: gnd -> GND
- U7 pad 23: -hv-1 -> power-VCC
- U7 pad 3: gnd -> GND
- U7 pad 37: -hv-1 -> power-VCC
- U7 pad 39: -hv-1 -> power-VCC
- U7 pad 40: -hv-1 -> power-VCC
- U7 pad 41: gnd -> GND
- U7 pad 5: -hv-1 -> power-VCC
- U7 pad 7: gnd -> GND
- U7 pad 8: -hv-1 -> power-VCC
- U8 pad 2: gnd -> GND
- U9 pad 2: gnd -> GND
- X1 pad 2: gnd -> GND
- X1 pad 4: gnd -> GND
Routing:
- net GND: track 0.00 -> 205.4 mm, vias 0 -> 42
- net gnd: track 199.2 -> 0.00 mm, vias 41 -> 0
- net power-VCC: track 0.00 -> 145.9 mm, vias 0 -> 10
- net -hv-1: track 144.5 -> 0.00 mm, vias 10 -> 0
- net RSTOUT_N: track 35.7 -> 38.2 mm
- net P70_IRQ: track 38.1 -> 40.4 mm
- net prev_button: track 49.8 -> 48.9 mm
- net nALERT_nBC_IRQ: track 73.6 -> 72.9 mm
- net ADDR_COMM: track 1.79 -> 1.05 mm
- net RESET: track 2.00 -> 1.37 mm
- added copper zone on F.Cu, net GND
- added copper zone on In1.Cu, net GND
- added copper zone on In2.Cu, net GND
- removed copper zone on F.Cu, net gnd
- removed copper zone on In1.Cu, net gnd
- removed copper zone on In2.Cu, net gnd
